File: ti99-psu.sch (KiCad schematic (older format))
At the start: 9 parts, among them J1 DC +12V IN, J2 -5V Regulator In, J3 +5V Regulator In, J4 -5V Regulator Out, J5 +5V Regulator Out, J6 TI-99/4A Power, SW1 SW_DPST

Commit message: V1 sent to production
Parts:
- SW1: footprint (none) -> Button_Switch_THT:SW_Slider_DPST
Connections:
- net GND: now also J4.2 (Pin_2), J5.2 (Pin_2)
Changed lines of the file:
@@
 F 0 "SW1" H 2600 2625 50  0000 C CNN
 F 1 "SW_DPST" H 2600 2534 50  0000 C CNN
-F 2 "" H 2600 2300 50  0001 C CNN
+F 2 "Button_Switch_THT:SW_Slider_DPST" H 2600 2300 50  0001 C CNN
 F 3 "~" H 2600 2300 50  0001 C CNN
 	1    2600 2300
@@
 	5850 2300 6350 2300
 Wire Wire Line
-	6350 2300 6350 3000
+	6350 2300 6350 2400
 Wire Wire Line
 	6350 3000 5850 3000
@@
 L power:GND #PWR0105
 U 1 1 5F9D8E0C
-P 7000 2650
-F 0 "#PWR0105" H 7000 2400 50  0001 C CNN
-F 1 "GND" H 7005 2477 50  0000 C CNN
-F 2 "" H 7000 2650 50  0001 C CNN
-F 3 "" H 7000 2650 50  0001 C CNN
-	1    7000 2650
-	1    0    0    -1
-$EndComp
-Wire Wire Line
-	7100 2400 7000 2400
-Wire Wire Line
-	7000 2400 7000 2650
+P 6350 3250
+F 0 "#PWR0105" H 6350 3000 50  0001 C CNN
+F 1 "GND" H 6355 3077 50  0000 C CNN
+F 2 "" H 6350 3250 50  0001 C CNN
+F 3 "" H 6350 3250 50  0001 C CNN
+	1    6350 3250
+	1    0    0    -1
+$EndComp
+Wire Wire Line
+	6350 3000 6350 3250
 Wire Wire Line
 	5850 2900 6450 2900
@@
 	0    -1   -1   0
 $EndComp
+Connection ~ 6350 2400
+Wire Wire Line
+	6350 2400 6350 3000
+Connection ~ 6350 3000
+Wire Wire Line
+	6350 2400 7100 2400
 $EndSCHEMATC
